File: pcb/frontpanel_pcb/frontpanel_pcb/frontpanel_pcb.kicad_pcb (KiCad board)
At the start: 2 copper layers, 158 x 40 mm, 18 parts, among them J1 Conn_02x06_Top_Bottom, Q1 BSS138, U1 291V1, U2 NHD-2.8-25664

Commit message: pcb
Parts:
- C1, Q1, R4, R5, R6, R7: moved to B.Cu
- moved R3 239.8 mm to (193.6, 89.0)
- moved R2 238.5 mm to (193.6, 91.5)
- moved R1 202.8 mm to (193.6, 94.1)
- moved C1 186.4 mm to (147.9, 67.3), turned to 180 degrees
- moved J1 152.9 mm to (45.0, 86.3), turned to 180 degrees
- moved R4 150.1 mm to (111.0, 67.3), turned to -90 degrees
- moved Q1 136.8 mm to (74.2, 85.1)
- moved R7 129.3 mm to (76.7, 80.0), turned to -90 degrees
- moved R6 122.4 mm to (69.1, 86.3), turned to 90 degrees
- moved R5 120.0 mm to (59.0, 80.0), turned to -90 degrees
Routing:
- net +3V3: track 0.00 -> 168.3 mm, vias 0 -> 3
- net /JA2: track 0.00 -> 147.7 mm
- net /JA3: track 0.00 -> 145.5 mm, vias 0 -> 1
- net /JA1: track 0.00 -> 143.8 mm
Other:
- board size 158 x 40 mm -> 165 x 40 mm
