File: pcb/frontpanel_pcb/frontpanel_pcb/frontpanel_pcb.sch (KiCad schematic (older format))
At the start: 14 parts, among them J1 Conn_02x06_Top_Bottom, Q1 BSS138, U1 291V1, U2 NHD-2.8-25664

Commit message: pcb
Parts:
- added C?: 10u, Capacitor_SMD:C_1206_3216Metric, symbol Device:C
- C1: footprint Capacitor_SMD:C_1210_3225Metric -> Capacitor_SMD:C_1206_3216Metric
Other:
- moved on the sheet: C1
Changed lines of the file:
@@
 L Device:C C1
 U 1 1 5DB93CC2
-P 3000 1850
-F 0 "C1" H 3115 1896 50  0000 L CNN
-F 1 "10u" H 3115 1805 50  0000 L CNN
-F 2 "Capacitor_SMD:C_1210_3225Metric" H 3038 1700 50  0001 C CNN
-F 3 "~" H 3000 1850 50  0001 C CNN
-	1    3000 1850
+P 4150 1300
+F 0 "C1" H 4265 1346 50  0000 L CNN
+F 1 "10u" H 4265 1255 50  0000 L CNN
+F 2 "Capacitor_SMD:C_1206_3216Metric" H 4188 1150 50  0001 C CNN
+F 3 "~" H 4150 1300 50  0001 C CNN
+	1    4150 1300
 	0    -1   -1   0
 $EndComp
@@
 L power:+3V3 #PWR0106
 U 1 1 5DB95488
-P 2850 1850
-F 0 "#PWR0106" H 2850 1700 50  0001 C CNN
-F 1 "+3V3" H 2865 2023 50  0000 C CNN
-F 2 "" H 2850 1850 50  0001 C CNN
-F 3 "" H 2850 1850 50  0001 C CNN
-	1    2850 1850
+P 4000 1300
+F 0 "#PWR0106" H 4000 1150 50  0001 C CNN
+F 1 "+3V3" H 4015 1473 50  0000 C CNN
+F 2 "" H 4000 1300 50  0001 C CNN
+F 3 "" H 4000 1300 50  0001 C CNN
+	1    4000 1300
 	0    -1   -1   0
 $EndComp
@@
 L power:GND #PWR0108
 U 1 1 5DB963FD
-P 3150 1850
-F 0 "#PWR0108" H 3150 1600 50  0001 C CNN
-F 1 "GND" H 3155 1677 50  0000 C CNN
-F 2 "" H 3150 1850 50  0001 C CNN
-F 3 "" H 3150 1850 50  0001 C CNN
-	1    3150 1850
+P 4300 1300
+F 0 "#PWR0108" H 4300 1050 50  0001 C CNN
+F 1 "GND" H 4305 1127 50  0000 C CNN
+F 2 "" H 4300 1300 50  0001 C CNN
+F 3 "" H 4300 1300 50  0001 C CNN
+	1    4300 1300
 	0    -1   -1   0
 $EndComp
@@
 Wire Wire Line
 	1100 2900 1700 2900
+$Comp
+L Device:C C?
+U 1 1 5DB8DE37
+P 4300 4350
+F 0 "C?" H 4415 4396 50  0000 L CNN
+F 1 "10u" H 4415 4305 50  0000 L CNN
+F 2 "Capacitor_SMD:C_1206_3216Metric" H 4338 4200 50  0001 C CNN
+F 3 "~" H 4300 4350 50  0001 C CNN
+	1    4300 4350
+	0    -1   -1   0
+$EndComp
+$Comp
+L power:+3V3 #PWR?
+U 1 1 5DB8DE48
+P 4150 4350
+F 0 "#PWR?" H 4150 4200 50  0001 C CNN
+F 1 "+3V3" H 4165 4523 50  0000 C CNN
+F 2 "" H 4150 4350 50  0001 C CNN
+F 3 "" H 4150 4350 50  0001 C CNN
+	1    4150 4350
+	0    -1   -1   0
+$EndComp
+$Comp
+L power:GND #PWR?
+U 1 1 5DB8DE56
+P 4450 4350
+F 0 "#PWR?" H 4450 4100 50  0001 C CNN
+F 1 "GND" H 4455 4177 50  0000 C CNN
+F 2 "" H 4450 4350 50  0001 C CNN
+F 3 "" H 4450 4350 50  0001 C CNN
+	1    4450 4350
+	0    -1   -1   0
+$EndComp
 $EndSCHEMATC
