File: hardware/frontpanel_pcb/frontpanel_pcb/frontpanel_pcb.sch (KiCad schematic (older format))
At the start: 15 parts, among them J1 Conn_02x06_Top_Bottom, Q1 BSS138, U1 291V1, U2 NHD-2.8-25664

Commit message: First PCB cut
Parts:
- gave numbers to parts that had none: 1
Connections:
- wire segments 39 -> 35
Changed lines of the file:
@@
 $EndComp
-Wire Wire Line
-	2200 2700 3500 2700
-Wire Wire Line
-	3500 2700 3500 2850
 Wire Wire Line
 	3500 2850 3800 2850
 Wire Wire Line
-	2200 2600 3550 2600
-Wire Wire Line
-	3550 2600 3550 2650
-Wire Wire Line
-	3550 2650 3800 2650
-Wire Wire Line
-	2200 2500 3550 2500
-Wire Wire Line
-	2200 2400 3500 2400
-Wire Wire Line
-	3500 2400 3500 2250
-Wire Wire Line
 	3500 2250 3800 2250
-Wire Wire Line
-	3800 2450 3550 2450
-Wire Wire Line
-	3550 2450 3550 2500
 $Comp
 L power:GND #PWR0109
@@
 Wire Wire Line
 	2800 4900 3200 4900
-Text Label 2900 4900 0    50   ~ 0
+Text Label 2900 5050 0    50   ~ 0
 JA1
-Text Label 2900 5050 0    50   ~ 0
+Text Label 2900 5200 0    50   ~ 0
 JA2
 $Comp
@@
 Wire Wire Line
 	3600 4500 3600 4550
-Text Label 2900 5200 0    50   ~ 0
+Text Label 2900 4900 0    50   ~ 0
 JA3
 Text Label 2300 2500 0    50   ~ 0
@@
 Wire Wire Line
 	1700 2600 1400 2600
-Text Label 2300 2700 0    50   ~ 0
-JA10
 $Comp
 L power:+3V3 #PWR0104
@@
 	1100 2900 1700 2900
 $Comp
-L Device:C C?
+L Device:C C2
 U 1 1 5DB8DE37
 P 4300 4350
-F 0 "C?" H 4415 4396 50  0000 L CNN
+F 0 "C2" H 4415 4396 50  0000 L CNN
 F 1 "10u" H 4415 4305 50  0000 L CNN
 F 2 "Capacitor_SMD:C_1206_3216Metric" H 4338 4200 50  0001 C CNN
@@
 $EndComp
 $Comp
-L power:+3V3 #PWR?
+L power:+3V3 #PWR0127
 U 1 1 5DB8DE48
 P 4150 4350
-F 0 "#PWR?" H 4150 4200 50  0001 C CNN
+F 0 "#PWR0127" H 4150 4200 50  0001 C CNN
 F 1 "+3V3" H 4165 4523 50  0000 C CNN
 F 2 "" H 4150 4350 50  0001 C CNN
@@
 $EndComp
 $Comp
-L power:GND #PWR?
+L power:GND #PWR0128
 U 1 1 5DB8DE56
 P 4450 4350
-F 0 "#PWR?" H 4450 4100 50  0001 C CNN
+F 0 "#PWR0128" H 4450 4100 50  0001 C CNN
 F 1 "GND" H 4455 4177 50  0000 C CNN
 F 2 "" H 4450 4350 50  0001 C CNN
@@
 	0    -1   -1   0
 $EndComp
+Text Label 2300 2700 0    50   ~ 0
+JA10
+Wire Wire Line
+	2200 2400 2500 2400
+Wire Wire Line
+	2200 2500 2500 2500
+Wire Wire Line
+	2200 2600 2500 2600
+Wire Wire Line
+	2200 2700 2500 2700
+Wire Wire Line
+	3500 2450 3800 2450
+Wire Wire Line
+	3500 2650 3800 2650
+Text Label 3600 2850 0    50   ~ 0
+JA7
+Text Label 3600 2450 0    50   ~ 0
+JA9
+Text Label 3600 2650 0    50   ~ 0
+JA10
+Text Label 3600 2250 0    50   ~ 0
+JA8
 $EndSCHEMATC
