File: hardware/si570_pmod/si570_pmod.kicad_pcb (KiCad board)
At the start: 2 copper layers, 40 x 20.3 mm, 17 parts, among them J1 Conn_01x06_Top_Bottom, J2 Conn_Coaxial, J3 Conn_Coaxial, J4 Conn_Coaxial, J5 Conn_Coaxial, U1 Si570

Commit message: pmod si570: add note about flipped J1
Other:
- board text added: "TODO: J1 is flipped !!!"
